File: fightpad-pcb.kicad_sch (KiCad schematic)
At the start: 13 parts, among them SW1 SW_PUSH, U1 ATmega32U4-A, Y1 16MHz

Commit message: Schematic Finished
Schematic finished with slight modifications. Further changes to be made, but this is the base version
Parts:
- added D1, D2, D3, D4: D_Small, Diode_SMD:D_SOD-123, symbol Device:D_Small
- added F1: Polyfuse, Fuse:Fuse_1206_3216Metric, symbol Device:Polyfuse
- added MX1, MX2, MX3, MX4: MX-NoLED, MX_Alps_Hybrid:MX-1U, symbol MX_Alps_Hybrid:MX-NoLED
- added USB1: Molex-0548190589, random-keyboard-parts:Molex-0548190589, symbol random-keyboard-parts:Molex-0548190589
- C1, C2, C3, C4, C5, C6: footprint (none) -> Capacitor_SMD:C_0805_2012Metric
- R1, R2, R3, R4: footprint (none) -> Resistor_SMD:R_0805_2012Metric
- SW1: footprint (none) -> random-keyboard-parts:SKQG-1155865
- Y1: footprint (none) -> Crystal:Crystal_SMD_3225-4Pin_3.2x2.5mm
Connections:
- net +5V: now also F1.1
- net D+: now also R2.2, USB1.3 (D+)
- net D-: now also USB1.4 (D-)
- net GND: now also USB1.1 (GND)
- net Row0: now reaches U1.27 (PD7)
- net Row0: now also D1.1 (K), D2.1 (K), D3.1 (K), D4.1 (K)
- net Col0: now reaches U1.28 (PB4)
- net Col0: now also MX1.1 (COL), MX2.1 (COL)
- net Col1: now reaches U1.29 (PB5)
- net Col1: now also MX3.1 (COL), MX4.1 (COL)
- new net: D4.2 (A), MX4.2 (ROW)
- new net: D2.2 (A), MX2.2 (ROW)
- new net: D1.2 (A), MX1.2 (ROW)
- new net: D3.2 (A), MX3.2 (ROW)
- new net VCC: F1.2, USB1.5 (VBUS)
